File: STP240320_0200B_b2b/STP240320_0200B_b2b.kicad_sch (KiCad schematic)
At the start: 2 parts, among them J1 Conn_02x08_Odd_Even

Commit message: ci: add CI (#1)
Other:
- title: (none) -> STP240320_0200B Board to Board Connector Adapter
Changed lines of the file:
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@@
 (kicad_sch (version 20211123) (generator eeschema)
   (paper "A4")
+  (title_block
+    (title "STP240320_0200B Board to Board Connector Adapter")
+    (date "${DATE}")
+    (rev "${TAG} (${REVISION})")
+  )
   (junction (at 96.52 60.96) (diameter 0) (color 0 0 0 0)
   )
