File: STP240320_0200B_b2b_breakout/STP240320_0200B_b2b_breakout.kicad_sch (KiCad schematic)
At the start: 18 parts, among them J1 Micro_SD_Card_Det_Hirose_DM3AT, J2 Conn_01x11, Q1 BSS138, U1 74HC4050D, U2 AP2112K-3.3, U3 LM809M3X-2.93

Commit message: all: cleanup revision info
Parts:
- LOGO1: footprint Symbol:OSHW-Symbol_6.7x6mm_SilkScreen -> Gigahawk:OSHW-Logo2_9.8x8mm_Mask
Changed lines of the file:
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@@
     (title "Breakout board for STP240320_0200B_b2b")
     (date "${DATE}")
-    (rev "${TAG} (${REVISION})")
+    (rev "${TAG} (${HASH})")
   )
   (junction (at 224.79 74.93) (diameter 0) (color 0 0 0 0)
@@
       (effects (font (size 1.27 1.27)) hide)
     )
-    (property "Footprint" "Symbol:OSHW-Symbol_6.7x6mm_SilkScreen" (at 269.24 156.21 0)
-      (effects (font (size 1.27 1.27)) hide)
-    )
+    (property "Footprint" "Gigahawk:OSHW-Logo2_9.8x8mm_Mask" (at 269.24 156.21 0)
+      (effects (font (size 1.27 1.27)) hide)
+    )
